Commit message: A variety of edits for quadrotor

File: configs/urdf/quadrotor_base.urdf.xacro (robot description, xacro)
@@ -19,5 +19,5 @@
         <origin xyz="0 0 -0.1" rpy="0 0 0" />
         <geometry>
-          <box size="0.2 0.2 0.18"/>
+          <box size="0.2 0.28 0.18"/>
         </geometry>
       </collision>
