Commit message: turtlebot working

File: configs/urdf/pioneer3at_simplified.xacro (robot description, xacro)
@@ -26,7 +26,7 @@
         </visual>
         <collision>
-            <origin xyz="-0.02 0 0.147" rpy="0 0 0"/>
+            <origin xyz="-0.02 0 0.167" rpy="0 0 0"/>
                 <geometry>
-                  <box size="0.54 0.5 0.26"/>
+                  <box size="0.54 0.5 0.22"/>
                 </geometry>
         </collision>
