Commit message: Got pioneer more or less working

File: configs/urdf/pioneer_realsense.xacro (robot description, xacro)
@@ -60,5 +60,5 @@
     </joint>
   <joint name="base_real" type="fixed">
-	<origin xyz="0.25 0 0.24" rpy="0 0 0"/>
+	<origin xyz="0.26 0 0.21" rpy="0 0 0"/>
 	<parent link="base_link"/>
 	<child link="rs200_camera"/>

Commit message: Moved realsense back so it doesn't end up in front of the hallucination. Should add a catch for that condition in the box geometry model

File: configs/urdf/pioneer_realsense.xacro (robot description, xacro)
@@ -60,5 +60,5 @@
     </joint>
   <joint name="base_real" type="fixed">
-	<origin xyz="0.26 0 0.21" rpy="0 0 0"/>
+	<origin xyz="0.24 0 0.21" rpy="0 0 0"/>
 	<parent link="base_link"/>
 	<child link="rs200_camera"/>

Commit message: Added bumper to pioneer chassis and temporarily reenabled local costmap for egocylindrical_pips_dwa (just for visualization purposes)

File: configs/urdf/pioneer_realsense.xacro (robot description, xacro)
@@ -178,3 +178,15 @@
         </sensor>
     </gazebo>
+    <gazebo reference="base_link">
+      <sensor name='bumper_contact' type='contact'>
+        <contact>
+          <collision>base_link_collision</collision>
+        </contact>
+        <update_rate> 5 </update_rate>
+        <plugin name="gripper_bumper" filename="libgazebo_ros_bumper.so">
+          <bumperTopicName>base_bumper</bumperTopicName>
+          <frameName>base_link</frameName>
+        </plugin>
+      </sensor>
+    </gazebo>
 </robot>

Commit message: Added bumpers to wheels of pioneer (only front work) and created script to publish bumper events

File: configs/urdf/pioneer_realsense.xacro (robot description, xacro)
@@ -179,5 +179,5 @@
     </gazebo>
     <gazebo reference="base_link">
-      <sensor name='bumper_contact' type='contact'>
+      <sensor name='base_link_bumper' type='contact'>
         <contact>
           <collision>base_link_collision</collision>
@@ -186,5 +186,53 @@
         <plugin name="gripper_bumper" filename="libgazebo_ros_bumper.so">
           <bumperTopicName>base_bumper</bumperTopicName>
-          <frameName>base_link</frameName>
+          <frameName>world</frameName>
+        </plugin>
+      </sensor>
+    </gazebo>
+    <gazebo reference="p3at_front_left_wheel">
+      <sensor name='p3at_front_left_wheel_bumper' type='contact'>
+        <contact>
+          <collision>p3at_front_left_wheel_collision</collision>
+        </contact>
+        <update_rate> 5 </update_rate>
+        <plugin name="p3at_front_left_wheel_bumper" filename="libgazebo_ros_bumper.so">
+          <bumperTopicName>base_bumper</bumperTopicName>
+          <frameName>world</frameName>
+        </plugin>
+      </sensor>
+    </gazebo>
+    <gazebo reference="p3at_front_right_wheel">
+      <sensor name='p3at_front_right_wheel_bumper' type='contact'>
+        <contact>
+          <collision>p3at_front_right_wheel_collision</collision>
+        </contact>
+        <update_rate> 5 </update_rate>
+        <plugin name="p3at_front_right_wheel_bumper" filename="libgazebo_ros_bumper.so">
+          <bumperTopicName>base_bumper</bumperTopicName>
+          <frameName>world</frameName>
+        </plugin>
+      </sensor>
+    </gazebo>
+    <gazebo reference="p3at_rear_left_wheel">
+      <sensor name='p3at_rear_left_wheel_bumper' type='contact'>
+        <contact>
+          <collision>p3at_rear_left_wheel_collision</collision>
+        </contact>
+        <update_rate> 5 </update_rate>
+        <plugin name="p3at_rear_left_wheel_bumper" filename="libgazebo_ros_bumper.so">
+          <bumperTopicName>base_bumper</bumperTopicName>
+          <frameName>world</frameName>
+        </plugin>
+      </sensor>
+    </gazebo>
+    <gazebo reference="p3at_rear_right_wheel">
+      <sensor name='p3at_rear_right_wheel_bumper' type='contact'>
+        <contact>
+          <collision>p3at_rear_right_wheel_collision</collision>
+        </contact>
+        <update_rate> 5 </update_rate>
+        <plugin name="p3at_rear_right_wheel_bumper" filename="libgazebo_ros_bumper.so">
+          <bumperTopicName>base_bumper</bumperTopicName>
+          <frameName>world</frameName>
         </plugin>
       </sensor>

Commit message: Fixed realsense incorrect frame_id issue

File: configs/urdf/pioneer_realsense.xacro (robot description, xacro)
@@ -33,4 +33,5 @@
     <!-- Virtual links representing the cameras positons and orientations-->
     <link name="color" />
+    <link name="color_frame" />
     <link name="depth" />
     <link name="ired1" />
@@ -43,4 +44,11 @@
         <!-- The default position is change since in Rviz the cloud depth axis is Z not X-->
         <origin xyz="0 -0.046 0.004" rpy="${pi/2} ${pi} ${pi/2}"/>
+    </joint>
+    <joint name="color_frame_joint" type="fixed">
+        <parent link="rs200_camera" />
+        <child link="color_frame" />
+        <!-- <origin xyz="0 -0.046 0.004" rpy="0 0 0"/> -->
+        <!-- The default position is change since in Rviz the cloud depth axis is Z not X-->
+        <origin xyz="0 -0.046 0.004" rpy="0 0 0"/>
     </joint>
     <joint name="depth_joint" type="fixed">
@@ -72,5 +80,5 @@
     </gazebo>
     <!-- Load parameters to model's main link-->
-    <gazebo reference="rs200_camera">
+    <gazebo reference="color_frame">
         <self_collide>0</self_collide>
         <enable_wind>0</enable_wind>
