Commit message: change params for pioneer

File: configs/robots/pioneer3at_simplified.xacro (robot description, xacro)
@@ -26,7 +26,7 @@
         </visual>
         <collision>
-            <origin xyz="0 0 0.217" rpy="0 0 0"/>
+            <origin xyz="0 0 0.227" rpy="0 0 0"/>
                 <geometry>
-                  <box size="0.62 0.48 0.28"/>
+                  <box size="0.64 0.54 0.3"/>
                 </geometry>
         </collision>
