Commit message: Added wheels to box-turtle

File: configs/robots/turtle_pioneer.urdf.xacro (robot description, xacro)
@@ -240,4 +240,198 @@
     <kobuki_sim/>
   </xacro:macro>
+  <!-- Front Axles + Wheels + Hubcaps -->
+  <xacro:macro name="p3at_front" params="suffix reflect">
+      <link name="p3at_front_${suffix}_axle">
+          <inertial>
+              <mass value="0.1"/>
+              <origin xyz="0 0 0"/>
+              <inertia ixx="1.0" ixy="0.0" ixz="0.0"
+                   iyy="1.0" iyz="0.0" izz="1.0"/>
+          </inertial>
+      <visual name="base_visual">
+          <origin xyz="0 0 0" rpy="0 0 0"/>
+          <geometry name="pioneer_geom">
+              <mesh filename="package://p3at_tutorial/meshes/p3at_meshes/axle.dae"/>
+          </geometry>
+          <material name="AxleGrey">
+              <color rgba="0.5 0.5 0.5 1"/>
+          </material>
+      </visual>
+      <collision>
+          <origin xyz="0 0 0" rpy="0 0 0"/>
+          <geometry>
+              <box size="0.01 0.01 0.01"/>
+          </geometry>
+      </collision>
+      </link>
+      <gazebo reference="p3at_front_${suffix}_axle">
+          <material value="Gazebo/Grey"/>
+      </gazebo>
+      <joint name="base_front_${suffix}_axle_joint" type="fixed">
+          <origin xyz="0.135 ${reflect*0.156} 0.111" rpy="0 0 0"/>
+          <parent link="base_link"/>
+          <child link="p3at_front_${suffix}_axle"/>
+      </joint>
+      <link name="p3at_front_${suffix}_hub">
+          <inertial>
+              <mass value="0.1"/>
+              <origin xyz="0 0 0"/>
+              <inertia ixx="1.0" ixy="0.0" ixz="0.0"
+                   iyy="1.0" iyz="0.0" izz="1.0"/>
+          </inertial>
+      <visual name="base_visual">
+          <origin xyz="0 0 0" rpy="0 0 0"/>
+          <geometry name="pioneer_geom">
+              <mesh filename="package://p3at_tutorial/meshes/p3at_meshes/${suffix}_hubcap.dae"/>
+          </geometry>
+          <material name="HubcapYellow">
+              <color rgba="1.0 0.811 0.151 1.0"/>
+          </material>
+      </visual>
+      <collision>
+          <origin xyz="0 0 0" rpy="0 0 0"/>
+          <geometry>
+              <box size="0.01 0.01 0.01"/>
+          </geometry>
+      </collision>
+      </link>
+      <gazebo reference="p3at_front_${suffix}_hub">
+          <material value="Gazebo/Yellow"/>
+      </gazebo>
+      <joint name="base_front_${suffix}_hub_joint" type="fixed">
+          <origin xyz="0 ${reflect*0.041} 0" rpy="0 0 0"/>
+          <parent link="p3at_front_${suffix}_axle"/>
+          <child link="p3at_front_${suffix}_hub"/>
+      </joint>
+      <link name="p3at_front_${suffix}_wheel">
+          <inertial>
+              <mass value="0.5"/>
+              <origin xyz="0 0 0"/>
+              <inertia ixx="0.012411765597" ixy="0" ixz="0"
+           iyy="0.015218160428" iyz="0" izz="0.011763977943"/>
+        </inertial>
+      <visual name="base_visual">
+          <origin xyz="0 0 0" rpy="0 0 0"/>
+          <geometry name="pioneer_geom">
+              <mesh filename="package://p3at_tutorial/meshes/p3at_meshes/wheel.dae"/>
+          </geometry>
+          <material name="WheelBlack">
+              <color rgba="0.117 0.117 0.117 1"/>
+          </material>
+      </visual>
+      <collision>
+          <origin xyz="0 0 0" rpy="${-3.1415927/2} 0 0"/>
+          <geometry>
+          <!--mesh filename="package://p3at_tutorial/meshes/p3at_meshes/wheel.dae"/-->
+          <cylinder radius="0.111" length="0.075"/>
+          </geometry>
+      </collision>
+      </link>
+      <gazebo reference="p3at_front_${suffix}_wheel">
+          <material value="Gazebo/Black"/>
+      </gazebo>
+      <joint name="p3at_front_${suffix}_wheel_joint" type="fixed">
+        <axis xyz="0 1 0"/>
+            <anchor xyz="0 0 0"/>
+        <origin xyz="0 0 0" rpy="0 0 0"/>
+        <parent link="p3at_front_${suffix}_hub"/>
+        <child link="p3at_front_${suffix}_wheel"/>
+      </joint>
+  <!-- Back Axles + Wheels + Hubcaps -->
+      <link name="p3at_back_${suffix}_axle">
+          <inertial>
+              <mass value="0.1"/>
+              <origin xyz="0 0 0"/>
+              <inertia ixx="1.0" ixy="0.0" ixz="0.0"
+                   iyy="1.0" iyz="0.0" izz="1.0"/>
+          </inertial>
+      <visual name="base_visual">
+          <origin xyz="0 0 0" rpy="0 0 0"/>
+          <geometry name="pioneer_geom">
+              <mesh filename="package://p3at_tutorial/meshes/p3at_meshes/axle.dae"/>
+          </geometry>
+          <material name="AxleGrey">
+              <color rgba="0.5 0.5 0.5 1"/>
+          </material>
+      </visual>
+      <collision>
+          <origin xyz="0 0 0" rpy="0 0 0"/>
+          <geometry>
+              <mesh filename="package://p3at_tutorial/meshes/p3at_meshes/axle.dae"/>
+          </geometry>
+      </collision>
+      </link>
+      <gazebo reference="p3at_back_${suffix}_axle">
+          <material value="Gazebo/Grey"/>
+      </gazebo>
+      <joint name="p3at_back_${suffix}_axle_joint" type="fixed">
+          <origin xyz="-0.134 ${reflect*0.156} 0.111" rpy="0 0 0"/>
+          <parent link="base_link"/>
+          <child link="p3at_back_${suffix}_axle"/>
+      </joint>
+      <link name="p3at_back_${suffix}_hub">
+          <inertial>
+              <mass value="0.1"/>
+              <origin xyz="0 0 0"/>
+              <inertia ixx="1.0" ixy="0.0" ixz="0.0"
+                   iyy="1.0" iyz="0.0" izz="1.0"/>
+          </inertial>
+      <visual name="base_visual">
+          <origin xyz="0 0 0" rpy="0 0 0"/>
+          <geometry name="pioneer_geom">
+              <mesh filename="package://p3at_tutorial/meshes/p3at_meshes/${suffix}_hubcap.dae"/>
+          </geometry>
+          <material name="HubcapYellow"/>
+      </visual>
+      <collision>
+          <origin xyz="0 0 0" rpy="0 0 0"/>
+          <geometry>
+              <mesh filename="package://p3at_tutorial/meshes/p3at_meshes/${suffix}_hubcap.dae"/>
+          </geometry>
+      </collision>
+      </link>
+      <gazebo reference="p3at_back_${suffix}_hub">
+          <material value="Gazebo/Yellow"/>
+      </gazebo>
+      <joint name="p3at_back_${suffix}_hub_joint" type="fixed">
+          <origin xyz="-0 ${reflect*0.041} 0" rpy="0 0 0"/>
+          <parent link="p3at_back_${suffix}_axle"/>
+          <child link="p3at_back_${suffix}_hub"/>
+      </joint>
+      <link name="p3at_back_${suffix}_wheel">
+          <inertial>
+              <mass value="0.5"/>
+              <origin xyz="0 0 0"/>
+              <inertia ixx="0.012411765597" ixy="0" ixz="0"
+           iyy="0.015218160428" iyz="0" izz="0.011763977943"/>
+        </inertial>
+      <visual name="base_visual">
+          <origin xyz="0 0 0" rpy="0 0 0"/>
+          <geometry name="pioneer_geom">
+              <mesh filename="package://p3at_tutorial/meshes/p3at_meshes/wheel.dae"/>
+          </geometry>
+          <material name="WheelBlack"/>
+      </visual>
+      <collision>
+          <origin xyz="0 0 0" rpy="${-3.1415927/2} 0 0"/>
+          <geometry>
+          <!--mesh filename="package://p3at_tutorial/meshes/p3at_meshes/wheel.dae"/-->
+          <cylinder radius="0.111" length="0.075"/>
+          </geometry>
+      </collision>
+      </link>
+      <gazebo reference="p3at_back_${suffix}_wheel">
+          <material value="Gazebo/Black"/>
+      </gazebo>
+      <joint name="p3at_back_${suffix}_wheel_joint" type="fixed">
+        <axis xyz="0 1 0"/>
+            <anchor xyz="0 0 0"/>
+          <origin xyz="0 0 0" rpy="0 0 0"/>
+          <parent link="p3at_back_${suffix}_hub"/>
+          <child link="p3at_back_${suffix}_wheel"/>
+      </joint>
+  </xacro:macro>
   <kobuki/>
+  <xacro:p3at_front suffix="left" reflect="1"/>
+  <xacro:p3at_front suffix="right" reflect="-1"/>
 </robot>

Commit message: Removed inertial properties of pioneer parts so that box-turtle handles like turtlebot

File: configs/robots/turtle_pioneer.urdf.xacro (robot description, xacro)
@@ -243,10 +243,10 @@
   <xacro:macro name="p3at_front" params="suffix reflect">
       <link name="p3at_front_${suffix}_axle">
-          <inertial>
+          <!-- <inertial>
               <mass value="0.1"/>
               <origin xyz="0 0 0"/>
               <inertia ixx="1.0" ixy="0.0" ixz="0.0"
                    iyy="1.0" iyz="0.0" izz="1.0"/>
-          </inertial>
+          </inertial> -->
       <visual name="base_visual">
           <origin xyz="0 0 0" rpy="0 0 0"/>
@@ -274,10 +274,10 @@
       </joint>
       <link name="p3at_front_${suffix}_hub">
-          <inertial>
+          <!-- <inertial>
               <mass value="0.1"/>
               <origin xyz="0 0 0"/>
               <inertia ixx="1.0" ixy="0.0" ixz="0.0"
                    iyy="1.0" iyz="0.0" izz="1.0"/>
-          </inertial>
+          </inertial> -->
       <visual name="base_visual">
           <origin xyz="0 0 0" rpy="0 0 0"/>
@@ -305,10 +305,10 @@
       </joint>
       <link name="p3at_front_${suffix}_wheel">
-          <inertial>
+          <!-- <inertial>
               <mass value="0.5"/>
               <origin xyz="0 0 0"/>
               <inertia ixx="0.012411765597" ixy="0" ixz="0"
            iyy="0.015218160428" iyz="0" izz="0.011763977943"/>
-        </inertial>
+        </inertial> -->
       <visual name="base_visual">
           <origin xyz="0 0 0" rpy="0 0 0"/>
@@ -340,10 +340,10 @@
   <!-- Back Axles + Wheels + Hubcaps -->
       <link name="p3at_back_${suffix}_axle">
-          <inertial>
+          <!--<inertial>
               <mass value="0.1"/>
               <origin xyz="0 0 0"/>
               <inertia ixx="1.0" ixy="0.0" ixz="0.0"
                    iyy="1.0" iyz="0.0" izz="1.0"/>
-          </inertial>
+          </inertial> -->
       <visual name="base_visual">
           <origin xyz="0 0 0" rpy="0 0 0"/>
@@ -371,10 +371,10 @@
       </joint>
       <link name="p3at_back_${suffix}_hub">
-          <inertial>
+          <!--<inertial>
               <mass value="0.1"/>
               <origin xyz="0 0 0"/>
               <inertia ixx="1.0" ixy="0.0" ixz="0.0"
                    iyy="1.0" iyz="0.0" izz="1.0"/>
-          </inertial>
+          </inertial>-->
       <visual name="base_visual">
           <origin xyz="0 0 0" rpy="0 0 0"/>
@@ -400,10 +400,10 @@
       </joint>
       <link name="p3at_back_${suffix}_wheel">
-          <inertial>
+          <!--<inertial>
               <mass value="0.5"/>
               <origin xyz="0 0 0"/>
               <inertia ixx="0.012411765597" ixy="0" ixz="0"
            iyy="0.015218160428" iyz="0" izz="0.011763977943"/>
-        </inertial>
+        </inertial>-->
       <visual name="base_visual">
           <origin xyz="0 0 0" rpy="0 0 0"/>

Commit message: Adding realsense to boxturtle model

File: configs/robots/turtle_pioneer.urdf.xacro (robot description, xacro)
@@ -435,3 +435,175 @@
   <xacro:p3at_front suffix="left" reflect="1"/>
   <xacro:p3at_front suffix="right" reflect="-1"/>
+   <!-- Camera link -->
+    <link name="rs200_camera">
+        <visual>
+            <origin rpy="0 0 0" xyz="0 0 0"/>
+            <geometry>
+                <mesh filename="package://realsense_gazebo_plugin/models/realsense_camera/meshes/realsense.dae"/>
+            </geometry>
+        </visual>
+        <collision>
+            <geometry>
+                <box size="0.0078 0.130 0.0192"/>
+            </geometry>
+        </collision>
+        <inertial>
+            <mass value="0.0615752"/>
+            <origin rpy="0 0 0" xyz="0 0 0"/>
+            <inertia ixx="9.108e-05"
+                     ixy="0"
+                     ixz="0"
+                     iyy="2.51e-06"
+                     iyz="0"
+                     izz="8.931e-05"
+            />
+        </inertial>
+    </link>
+    <!-- Virtual links representing the cameras positons and orientations-->
+    <link name="color" />
+    <link name="depth" />
+    <link name="ired1" />
+    <link name="ired2" />
+    <!-- Joints positioning the virtual links with respect to the camera main link-->
+    <joint name="color_joint" type="fixed">
+        <parent link="rs200_camera" />
+        <child link="color" />
+        <!-- <origin xyz="0 -0.046 0.004" rpy="0 0 0"/> -->
+        <!-- The default position is change since in Rviz the cloud depth axis is Z not X-->
+        <origin xyz="0 -0.046 0.004" rpy="${pi/2} ${pi} ${pi/2}"/>
+    </joint>
+    <joint name="depth_joint" type="fixed">
+        <parent link="rs200_camera" />
+        <child link="depth" />
+        <origin xyz="0 -0.03 0.004" rpy="0 0 0"/>
+    </joint>
+    <joint name="ired1_joint" type="fixed">
+        <parent link="rs200_camera" />
+        <child link="ired1" />
+        <origin xyz="0 -0.06 0.004" rpy="0 0 0"/>
+    </joint>
+    <joint name="ired2_joint" type="fixed">
+        <parent link="rs200_camera" />
+        <child link="ired2" />
+        <origin xyz="0 0.01 0.004" rpy="0 0 0"/>
+    </joint>
+  <joint name="base_real" type="fixed">
+	<origin xyz="0.25 0 0.24" rpy="0 0 0"/>
+	<parent link="base_link"/>
+	<child link="rs200_camera"/>
+  </joint>
+<!-- **********************************************************-->
+<!-- GAZEBO DEFINITIONS ***************************************-->
+    <!-- Load plugin to the model ("robot" in urdf format)-->
+    <gazebo>
+        <plugin name="realsense_plugin" filename="librealsense_gazebo_plugin.so"/>
+        <!--<pose frame="">0 0 0.015 0 0 0</pose>-->
+    </gazebo>
+    <!-- Load parameters to model's main link-->
+    <gazebo reference="rs200_camera">
+        <self_collide>0</self_collide>
+        <enable_wind>0</enable_wind>
+        <kinematic>0</kinematic>
+        <gravity>1</gravity>
+        <!--<mu>1</mu>-->
+        <mu2>1</mu2>
+        <fdir1>0 0 0</fdir1>
+        <!--<slip1>0</slip1>
+        <slip2>0</slip2>-->
+        <kp>1e+13</kp>
+        <kd>1</kd>
+        <!--<max_vel>0.01</max_vel>
+        <min_depth>0</min_depth>-->
+        <sensor name="color" type="camera">
+            <pose frame="">0 -0.046 0.004 0 0 0</pose>
+            <camera name="__default__">
+            <horizontal_fov>1.047</horizontal_fov>
+            <image>
+                <width>640</width>
+                <height>480</height>
+                <format>RGB_INT8</format>
+            </image>
+            <clip>
+                <near>0.1</near>
+                <far>100</far>
+            </clip>
+            <noise>
+                <type>gaussian</type>
+                <mean>0.0</mean>
+                <stddev>0.007</stddev>
+            </noise>
+            </camera>
+            <always_on>1</always_on>
+            <update_rate>60</update_rate>
+            <visualize>1</visualize>
+        </sensor>
+        <sensor name="ired1" type="camera">
+            <pose frame="">0 -0.06 0.004 0 0 0</pose>
+            <camera name="__default__">
+            <horizontal_fov>1.047</horizontal_fov>
+            <image>
+                <width>640</width>
+                <height>480</height>
+                <format>L_INT8</format>
+            </image>
+            <clip>
+                <near>0.1</near>
+                <far>100</far>
+            </clip>
+            <noise>
+                <type>gaussian</type>
+                <mean>0.0</mean>
+                <stddev>0.05</stddev>
+            </noise>
+            </camera>
+            <always_on>1</always_on>
+            <update_rate>60</update_rate>
+            <visualize>0</visualize>
+        </sensor>
+        <sensor name="ired2" type="camera">
+            <pose frame="">0 0.01 0.004 0 0 0</pose>
+            <camera name="__default__">
+            <horizontal_fov>1.047</horizontal_fov>
+            <image>
+                <width>640</width>
+                <height>480</height>
+                <format>L_INT8</format>
+            </image>
+            <clip>
+                <near>0.1</near>
+                <far>100</far>
+            </clip>
+            <noise>
+                <type>gaussian</type>
+                <mean>0.0</mean>
+                <stddev>0.05</stddev>
+            </noise>
+            </camera>
+            <always_on>1</always_on>
+            <update_rate>60</update_rate>
+            <visualize>0</visualize>
+        </sensor>
+        <sensor name="depth" type="depth">
+            <pose frame="">0 -0.03 0.004 0 0 0</pose>
+            <camera name="__default__">
+            <horizontal_fov>1.047</horizontal_fov>
+            <image>
+                    <width>640</width>
+                    <height>480</height>
+            </image>
+            <clip>
+                    <near>0.1</near>
+                    <far>100</far>
+            </clip>
+            <noise>
+                    <type>gaussian</type>
+                    <mean>0.0</mean>
+                    <stddev>0.100</stddev>
+            </noise>
+            </camera>
+            <always_on>1</always_on>
+            <update_rate>60</update_rate>
+            <visualize>0</visualize>
+        </sensor>
+    </gazebo>
 </robot>
