Commit message: Hopefully functional box turtle

File: configs/robots/turtle_pioneer.urdf.xacro (robot description, xacro)
@@ -435,175 +435,4 @@
   <xacro:p3at_front suffix="left" reflect="1"/>
   <xacro:p3at_front suffix="right" reflect="-1"/>
-   <!-- Camera link -->
-    <link name="rs200_camera">
-        <visual>
-            <origin rpy="0 0 0" xyz="0 0 0"/>
-            <geometry>
-                <mesh filename="package://realsense_gazebo_plugin/models/realsense_camera/meshes/realsense.dae"/>
-            </geometry>
-        </visual>
-        <collision>
-            <geometry>
-                <box size="0.0078 0.130 0.0192"/>
-            </geometry>
-        </collision>
-        <inertial>
-            <mass value="0.0615752"/>
-            <origin rpy="0 0 0" xyz="0 0 0"/>
-            <inertia ixx="9.108e-05"
-                     ixy="0"
-                     ixz="0"
-                     iyy="2.51e-06"
-                     iyz="0"
-                     izz="8.931e-05"
-            />
-        </inertial>
-    </link>
-    <!-- Virtual links representing the cameras positons and orientations-->
-    <link name="color" />
-    <link name="depth" />
-    <link name="ired1" />
-    <link name="ired2" />
-    <!-- Joints positioning the virtual links with respect to the camera main link-->
-    <joint name="color_joint" type="fixed">
-        <parent link="rs200_camera" />
-        <child link="color" />
-        <!-- <origin xyz="0 -0.046 0.004" rpy="0 0 0"/> -->
-        <!-- The default position is change since in Rviz the cloud depth axis is Z not X-->
-        <origin xyz="0 -0.046 0.004" rpy="${pi/2} ${pi} ${pi/2}"/>
-    </joint>
-    <joint name="depth_joint" type="fixed">
-        <parent link="rs200_camera" />
-        <child link="depth" />
-        <origin xyz="0 -0.03 0.004" rpy="0 0 0"/>
-    </joint>
-    <joint name="ired1_joint" type="fixed">
-        <parent link="rs200_camera" />
-        <child link="ired1" />
-        <origin xyz="0 -0.06 0.004" rpy="0 0 0"/>
-    </joint>
-    <joint name="ired2_joint" type="fixed">
-        <parent link="rs200_camera" />
-        <child link="ired2" />
-        <origin xyz="0 0.01 0.004" rpy="0 0 0"/>
-    </joint>
-  <joint name="base_real" type="fixed">
-	<origin xyz="0.25 0 0.24" rpy="0 0 0"/>
-	<parent link="base_link"/>
-	<child link="rs200_camera"/>
-  </joint>
-<!-- **********************************************************-->
-<!-- GAZEBO DEFINITIONS ***************************************-->
-    <!-- Load plugin to the model ("robot" in urdf format)-->
-    <gazebo>
-        <plugin name="realsense_plugin" filename="librealsense_gazebo_plugin.so"/>
-        <!--<pose frame="">0 0 0.015 0 0 0</pose>-->
-    </gazebo>
-    <!-- Load parameters to model's main link-->
-    <gazebo reference="rs200_camera">
-        <self_collide>0</self_collide>
-        <enable_wind>0</enable_wind>
-        <kinematic>0</kinematic>
-        <gravity>1</gravity>
-        <!--<mu>1</mu>-->
-        <mu2>1</mu2>
-        <fdir1>0 0 0</fdir1>
-        <!--<slip1>0</slip1>
-        <slip2>0</slip2>-->
-        <kp>1e+13</kp>
-        <kd>1</kd>
-        <!--<max_vel>0.01</max_vel>
-        <min_depth>0</min_depth>-->
-        <sensor name="color" type="camera">
-            <pose frame="">0 -0.046 0.004 0 0 0</pose>
-            <camera name="__default__">
-            <horizontal_fov>1.047</horizontal_fov>
-            <image>
-                <width>640</width>
-                <height>480</height>
-                <format>RGB_INT8</format>
-            </image>
-            <clip>
-                <near>0.1</near>
-                <far>100</far>
-            </clip>
-            <noise>
-                <type>gaussian</type>
-                <mean>0.0</mean>
-                <stddev>0.007</stddev>
-            </noise>
-            </camera>
-            <always_on>1</always_on>
-            <update_rate>60</update_rate>
-            <visualize>1</visualize>
-        </sensor>
-        <sensor name="ired1" type="camera">
-            <pose frame="">0 -0.06 0.004 0 0 0</pose>
-            <camera name="__default__">
-            <horizontal_fov>1.047</horizontal_fov>
-            <image>
-                <width>640</width>
-                <height>480</height>
-                <format>L_INT8</format>
-            </image>
-            <clip>
-                <near>0.1</near>
-                <far>100</far>
-            </clip>
-            <noise>
-                <type>gaussian</type>
-                <mean>0.0</mean>
-                <stddev>0.05</stddev>
-            </noise>
-            </camera>
-            <always_on>1</always_on>
-            <update_rate>60</update_rate>
-            <visualize>0</visualize>
-        </sensor>
-        <sensor name="ired2" type="camera">
-            <pose frame="">0 0.01 0.004 0 0 0</pose>
-            <camera name="__default__">
-            <horizontal_fov>1.047</horizontal_fov>
-            <image>
-                <width>640</width>
-                <height>480</height>
-                <format>L_INT8</format>
-            </image>
-            <clip>
-                <near>0.1</near>
-                <far>100</far>
-            </clip>
-            <noise>
-                <type>gaussian</type>
-                <mean>0.0</mean>
-                <stddev>0.05</stddev>
-            </noise>
-            </camera>
-            <always_on>1</always_on>
-            <update_rate>60</update_rate>
-            <visualize>0</visualize>
-        </sensor>
-        <sensor name="depth" type="depth">
-            <pose frame="">0 -0.03 0.004 0 0 0</pose>
-            <camera name="__default__">
-            <horizontal_fov>1.047</horizontal_fov>
-            <image>
-                    <width>640</width>
-                    <height>480</height>
-            </image>
-            <clip>
-                    <near>0.1</near>
-                    <far>100</far>
-            </clip>
-            <noise>
-                    <type>gaussian</type>
-                    <mean>0.0</mean>
-                    <stddev>0.100</stddev>
-            </noise>
-            </camera>
-            <always_on>1</always_on>
-            <update_rate>60</update_rate>
-            <visualize>0</visualize>
-        </sensor>
-    </gazebo>
+  <xacro:include filename="$(find nav_configs)/urdf/pioneer_realsense.xacro" />
 </robot>

Commit message: box turtle is working now

File: configs/robots/turtle_pioneer.urdf.xacro (robot description, xacro)
@@ -62,5 +62,5 @@
         </inertial>
         <visual name="base_visual">
-            <origin xyz="0 0 0" rpy="0 0 0"/>
+            <origin xyz="0.01 0 0" rpy="0 0 0"/>
             <geometry name="pioneer_geom">
                 <mesh filename="package://p3at_tutorial/meshes/p3at_meshes/top.dae"/>
@@ -71,7 +71,8 @@
         </visual>
         <collision>
-            <origin xyz="0 0 0" rpy="0 0 0"/>
+            <origin xyz="0.01 0 0" rpy="0 0 0"/>
             <geometry>
-                <box size="0.01 0.01 0.01"/>
+		<mesh filename="package://p3at_tutorial/meshes/p3at_meshes/top.dae"/>
+                <!--<box size="0.01 0.01 0.01"/>-->
             </geometry>
         </collision>
@@ -81,5 +82,5 @@
     </gazebo>
     <joint name="base_top_joint" type="fixed">
-        <origin xyz="0.003 0 0.274" rpy="0 0 0"/>
+        <origin xyz="0.028 0 0.274" rpy="0 0 0"/>
         <parent link="base_link"/>
         <child link="top_plate"/>
@@ -243,6 +244,6 @@
   <xacro:macro name="p3at_front" params="suffix reflect">
       <link name="p3at_front_${suffix}_axle">
-          <!-- <inertial>
-              <mass value="0.1"/>
+          <!--<inertial>
+              <mass value="0.001"/>
               <origin xyz="0 0 0"/>
               <inertia ixx="1.0" ixy="0.0" ixz="0.0"
@@ -274,10 +275,10 @@
       </joint>
       <link name="p3at_front_${suffix}_hub">
-          <!-- <inertial>
-              <mass value="0.1"/>
+          <!--<inertial>
+              <mass value="0.001"/>
               <origin xyz="0 0 0"/>
               <inertia ixx="1.0" ixy="0.0" ixz="0.0"
                    iyy="1.0" iyz="0.0" izz="1.0"/>
-          </inertial> -->
+          </inertial>-->
       <visual name="base_visual">
           <origin xyz="0 0 0" rpy="0 0 0"/>
@@ -305,10 +306,10 @@
       </joint>
       <link name="p3at_front_${suffix}_wheel">
-          <!-- <inertial>
-              <mass value="0.5"/>
+          <!--<inertial>
+              <mass value="0.001"/>
               <origin xyz="0 0 0"/>
               <inertia ixx="0.012411765597" ixy="0" ixz="0"
            iyy="0.015218160428" iyz="0" izz="0.011763977943"/>
-        </inertial> -->
+        </inertial>-->
       <visual name="base_visual">
           <origin xyz="0 0 0" rpy="0 0 0"/>
@@ -341,9 +342,9 @@
       <link name="p3at_back_${suffix}_axle">
           <!--<inertial>
-              <mass value="0.1"/>
+              <mass value="0.001"/>
               <origin xyz="0 0 0"/>
               <inertia ixx="1.0" ixy="0.0" ixz="0.0"
                    iyy="1.0" iyz="0.0" izz="1.0"/>
-          </inertial> -->
+          </inertial>-->
       <visual name="base_visual">
           <origin xyz="0 0 0" rpy="0 0 0"/>
@@ -372,5 +373,5 @@
       <link name="p3at_back_${suffix}_hub">
           <!--<inertial>
-              <mass value="0.1"/>
+              <mass value="0.001"/>
               <origin xyz="0 0 0"/>
               <inertia ixx="1.0" ixy="0.0" ixz="0.0"
@@ -401,5 +402,5 @@
       <link name="p3at_back_${suffix}_wheel">
           <!--<inertial>
-              <mass value="0.5"/>
+              <mass value="0.001"/>
               <origin xyz="0 0 0"/>
               <inertia ixx="0.012411765597" ixy="0" ixz="0"

File: configs/urdf/pioneer3at_simplified.xacro (robot description, xacro)
@@ -28,5 +28,5 @@
             <origin xyz="-0.02 0 0.167" rpy="0 0 0"/>
                 <geometry>
-                  <box size="0.54 0.5 0.22"/>
+                  <box size="0.56 0.5 0.22"/>
                 </geometry>
         </collision>
@@ -77,111 +77,4 @@
         <child link="top_plate"/>
     </joint>
-<!-- Front + Back Sonar -->
-    <link name="front_sonar">
-        <inertial>
-            <mass value="0.1"/>
-            <origin xyz="0 0 0"/>
-            <inertia ixx="1.0" ixy="0.0" ixz="0.0"
-                 iyy="1.0" iyz="0.0" izz="1.0"/>
-        </inertial>
-        <visual name="base_visual">
-            <origin xyz="0 0 0" rpy="0 0 0"/>
-            <geometry name="pioneer_geom">
-                <mesh filename="package://p3at_tutorial/meshes/p3at_meshes/front_sonar.dae"/>
-            </geometry>
-            <material name="SonarYellow">
-                <color rgba="0.715 0.583 0.210 1.0"/>
-            </material>
-        </visual>
-    </link>
-    <gazebo reference="front_sonar">
-        <material value="Gazebo/Yellow"/>
-    </gazebo>
-    <joint name="base_front_joint" type="fixed">
-        <origin xyz="0.193 0 0.25" rpy="0 0 0"/>
-        <parent link="base_link"/>
-        <child link="front_sonar"/>
-    </joint>
-    <link name="back_sonar">
-        <inertial>
-            <mass value="0.1"/>
-            <origin xyz="0 0 0"/>
-            <inertia ixx="1.0" ixy="0.0" ixz="0.0"
-                 iyy="1.0" iyz="0.0" izz="1.0"/>
-        </inertial>
-        <visual name="base_visual">
-            <origin xyz="0 0 0" rpy="0 0 0"/>
-            <geometry name="pioneer_geom">
-                <mesh filename="package://p3at_tutorial/meshes/p3at_meshes/back_sonar.dae"/>
-            </geometry>
-            <material name="SonarYellow">
-                <color rgba="0.715 0.583 0.210 1.0"/>
-            </material>
-        </visual>
-    </link>
-    <gazebo reference="back_sonar">
-        <material value="Gazebo/Yellow"/>
-    </gazebo>
-    <joint name="base_back_joint" type="fixed">
-        <origin xyz="-0.187 0 0.247" rpy="0 0 0"/>
-        <parent link="base_link"/>
-        <child link="back_sonar"/>
-    </joint>
-<link name="back_sonar_fake">
-    <inertial>
-            <mass value="0.1"/>
-            <origin xyz="0 0 0"/>
-            <inertia ixx="1.0" ixy="0.0" ixz="0.0"
-                 iyy="1.0" iyz="0.0" izz="1.0"/>
-    </inertial>
-<!--     <visual name="base_visual">
-            <origin xyz="0 0 0" rpy="0 0 0"/>
-            <geometry name="pioneer_geom">
-                <mesh filename="package://p3at_tutorial/meshes/p3at_meshes/back_sonar.dae"/>
-            </geometry>
-            <material name="SonarYellow">
-                <color rgba="0.715 0.583 0.210 1.0"/>
-            </material>
-        </visual>
-        <collision>
-            <origin xyz="0 0 0" rpy="0 0 0"/>
-            <geometry>
-                <box size="0.01 0.01 0.01"/>
-            </geometry>
-        </collision> -->
-</link>
-<joint name="base_back_sonar_joint" type="fixed">
-    <origin xyz="0 0 0" rpy="0 0 3.1415"/>
-    <parent link="back_sonar"/>
-    <child link="back_sonar_fake"/>
-</joint>
-<link name="imu">
-    <inertial>
-            <mass value="0.1"/>
-            <origin xyz="0 0 0"/>
-            <inertia ixx="1.0" ixy="0.0" ixz="0.0"
-                 iyy="1.0" iyz="0.0" izz="1.0"/>
-    </inertial>
-<!--     <visual name="base_visual">
-            <origin xyz="0 0 0" rpy="0 0 0"/>
-            <geometry name="pioneer_geom">
-                <mesh filename="package://p3at_tutorial/meshes/p3at_meshes/back_sonar.dae"/>
-            </geometry>
-            <material name="SonarYellow">
-                <color rgba="0.715 0.583 0.210 1.0"/>
-            </material>
-        </visual>
-        <collision>
-            <origin xyz="0 0 0" rpy="0 0 0"/>
-            <geometry>
-                <box size="0.01 0.01 0.01"/>
-            </geometry>
-        </collision> -->
-</link>
-<joint name="imu_joint" type="fixed">
-    <origin xyz="0 0 0" rpy="3.1415 0 0"/>
-    <parent link="base_link"/>
-    <child link="imu"/>
-</joint>
 <!-- Front Axles + Wheels + Hubcaps -->
 <xacro:macro name="p3at_front" params="suffix reflect">

File: configs/urdf/pioneer_realsense.xacro (robot description, xacro)
@@ -20,5 +20,5 @@
         </collision>
         <inertial>
-            <mass value="0.0615752"/>
+            <mass value="0.001"/>
             <origin rpy="0 0 0" xyz="0 0 0"/>
             <inertia ixx="9.108e-05"
@@ -180,9 +180,23 @@
     <gazebo reference="base_link">
       <sensor name='base_link_bumper' type='contact'>
-        <contact>
-          <collision>base_link_collision</collision>
-        </contact>
-        <update_rate> 5 </update_rate>
-        <plugin name="gripper_bumper" filename="libgazebo_ros_bumper.so">
+	<always_on>true</always_on>
+        <contact>
+          <collision>base_footprint_fixed_joint_lump__base_link_collision</collision>
+        </contact>
+        <update_rate> 5 </update_rate>
+        <plugin name="grimpper" filename="libgazebo_ros_bumper.so">
+          <bumperTopicName>base_bumper</bumperTopicName>
+          <frameName>world</frameName>
+        </plugin>
+      </sensor>
+    </gazebo>
+    <gazebo reference="top_plate">
+      <sensor name='top_plate_bumper' type='contact'>
+	<always_on>true</always_on>
+        <contact>
+          <collision>base_footprint_fixed_joint_lump__top_plate_collision_8</collision>
+        </contact>
+        <update_rate> 5 </update_rate>
+        <plugin name="top_plate_bumper" filename="libgazebo_ros_bumper.so">
           <bumperTopicName>base_bumper</bumperTopicName>
           <frameName>world</frameName>
@@ -192,6 +206,7 @@
     <gazebo reference="p3at_front_left_wheel">
       <sensor name='p3at_front_left_wheel_bumper' type='contact'>
-        <contact>
-          <collision>p3at_front_left_wheel_collision</collision>
+	<always_on>true</always_on>
+        <contact>
+          <collision>base_footprint_fixed_joint_lump__p3at_front_left_wheel_collision_3</collision>
         </contact>
         <update_rate> 5 </update_rate>
@@ -204,6 +219,7 @@
     <gazebo reference="p3at_front_right_wheel">
       <sensor name='p3at_front_right_wheel_bumper' type='contact'>
-        <contact>
-          <collision>p3at_front_right_wheel_collision</collision>
+	<always_on>true</always_on>
+        <contact>
+          <collision>base_footprint_fixed_joint_lump__p3at_front_right_wheel_collision_6</collision>
         </contact>
         <update_rate> 5 </update_rate>
@@ -214,23 +230,23 @@
       </sensor>
     </gazebo>
-    <gazebo reference="p3at_rear_left_wheel">
-      <sensor name='p3at_rear_left_wheel_bumper' type='contact'>
-        <contact>
-          <collision>p3at_rear_left_wheel_collision</collision>
-        </contact>
-        <update_rate> 5 </update_rate>
-        <plugin name="p3at_rear_left_wheel_bumper" filename="libgazebo_ros_bumper.so">
-          <bumperTopicName>base_bumper</bumperTopicName>
-          <frameName>world</frameName>
-        </plugin>
-      </sensor>
-    </gazebo>
-    <gazebo reference="p3at_rear_right_wheel">
-      <sensor name='p3at_rear_right_wheel_bumper' type='contact'>
-        <contact>
-          <collision>p3at_rear_right_wheel_collision</collision>
-        </contact>
-        <update_rate> 5 </update_rate>
-        <plugin name="p3at_rear_right_wheel_bumper" filename="libgazebo_ros_bumper.so">
+    <gazebo reference="p3at_back_left_wheel">
+      <sensor name='p3at_back_left_wheel_bumper' type='contact'>
+        <contact>
+          <collision>base_footprint_fixed_joint_lump__p3at_back_left_wheel_collision_13</collision>
+        </contact>
+        <update_rate> 5 </update_rate>
+        <plugin name="p3at_back_left_wheel_bumper" filename="libgazebo_ros_bumper.so">
+          <bumperTopicName>base_bumper</bumperTopicName>
+          <frameName>world</frameName>
+        </plugin>
+      </sensor>
+    </gazebo>
+    <gazebo reference="p3at_back_right_wheel">
+      <sensor name='p3at_back_right_wheel_bumper' type='contact'>
+        <contact>
+          <collision>base_footprint_fixed_joint_lump__p3at_back_right_wheel_collision_16</collision>
+        </contact>
+        <update_rate> 5 </update_rate>
+        <plugin name="p3at_back_right_wheel_bumper" filename="libgazebo_ros_bumper.so">
           <bumperTopicName>base_bumper</bumperTopicName>
           <frameName>world</frameName>

Commit message: Improved configurations for localization.

File: configs/robots/turtle_pioneer.urdf.xacro (robot description, xacro)
@@ -8,5 +8,5 @@
 <robot name="turtle_pioneer" xmlns:xacro="http://ros.org/wiki/xacro">
   <xacro:include filename="$(find kobuki_description)/urdf/common_properties.urdf.xacro"/>
-  <xacro:include filename="$(find kobuki_description)/urdf/kobuki_gazebo.urdf.xacro"/>
+  <xacro:include filename="$(find nav_configs)/urdf/kobuki_gazebo_gps.urdf.xacro"/>
   <!-- Kobuki -->
   <xacro:macro name="kobuki">
@@ -437,10 +437,3 @@
   <xacro:p3at_front suffix="right" reflect="-1"/>
   <xacro:include filename="$(find nav_configs)/urdf/pioneer_realsense.xacro" />
-  <gazebo>
-    <plugin name='gps_sensor' filename='libhector_gazebo_ros_gps.so'>
-      <updateRate>1</updateRate>
-      <bodyName>top_plate</bodyName>
-      <frameId>top_plate</frameId>
-    </plugin>
-  </gazebo>
 </robot>

File: configs/urdf/pioneer3at_simplified.xacro (robot description, xacro)
@@ -28,5 +28,5 @@
             <origin xyz="-0.02 0 0.167" rpy="0 0 0"/>
                 <geometry>
-                  <box size="0.56 0.5 0.22"/>
+                  <box size="0.56 0.4 0.22"/> <!-- "0.56 0.5 0.22" -->
                 </geometry>
         </collision>
