Commit message: modified for stereo

File: configs/turtlebot_stereo/camera.urdf.xacro (robot description, xacro)
@@ -1,10 +1,10 @@
 <?xml version="1.0"?>
 <robot name="sensor_camera" xmlns:xacro="http://ros.org/wiki/xacro">
-  <xacro:include filename="$(find sparse_stereo)/turtlebot_stereo/turtlebot_gazebo.urdf.xacro"/>
+  <xacro:include filename="$(find nav_configs)/turtlebot_stereo/turtlebot_gazebo.urdf.xacro"/>
   <xacro:include filename="$(find turtlebot_description)/urdf/turtlebot_properties.urdf.xacro"/>
   <!-- Hokuyo 2D LIDAR -->
   <xacro:macro name="sensor_camera" params="parent">
     <joint name="additional_camera" type="fixed">
-      <origin xyz="0.1 0.0 0.41" rpy="${cam_or} ${cam_op} ${cam_oy}" />
+      <origin xyz="0.1 0.0 0.2" rpy="${cam_or} ${cam_op} ${cam_oy}" />
       <parent link="base_link" />
       <child link="stereo_camera_frame" />

File: configs/turtlebot_stereo/kobuki_hexagons_kinect_stereo_camera.urdf.xacro (robot description, xacro)
@@ -11,5 +11,5 @@
   <xacro:include filename="$(find turtlebot_description)/urdf/stacks/hexagons.urdf.xacro"/>
   <xacro:include filename="$(find turtlebot_description)/urdf/sensors/kinect.urdf.xacro"/>
-  <xacro:include filename="$(find sparse_stereo)/turtlebot_stereo/camera.urdf.xacro"/>
+  <xacro:include filename="$(find nav_configs)/turtlebot_stereo/camera.urdf.xacro"/>
   <kobuki/>
   <stack_hexagons parent="base_link"/>

File: configs/turtlebot_stereo/turtlebot_gazebo.urdf.xacro (robot description, xacro)
@@ -49,10 +49,10 @@
             <width>640</width>
             <height>480</height>
-            <format>L8</format>
-            <!--format>R8G8B8</format-->
+            <!--<format>L8</format>-->
+            <format>B8G8R8</format>
           </image>
           <clip>
             <near>0.1</near>
-            <far>8</far>
+            <far>20</far>
           </clip>
           <noise>
@@ -68,10 +68,10 @@
             <width>640</width>
             <height>480</height>
-            <format>L8</format>
-            <!--format>R8G8B8</format-->
+            <!--<format>L8</format>-->
+            <format>B8G8R8</format>
           </image>
           <clip>
             <near>0.1</near>
-            <far>8</far>
+            <far>20</far>
           </clip>
           <noise>
